File: plans/schematic/Verdrahtungsplan.sch (EAGLE design)
At the start: 17 parts, among them J1 Buchse DC Hohlstecker, U1 NUCLEO-F401RE

Commit message: led library documetation, tests added; drawings
Connections:
- net MATRIX_DATA: now also U1G$2.PB15; no longer U1G$1.PA15
Changed lines of the file:
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@@
 <setting verticaltext="up"/>
 </settings>
-<grid distance="0.1" unitdist="inch" unit="inch" style="lines" multiple="1" display="yes" altdistance="0.01" altunitdist="inch" altunit="inch"/>
+<grid distance="0.1" unitdist="inch" unit="inch" style="lines" multiple="1" display="no" altdistance="0.01" altunitdist="inch" altunit="inch"/>
 <layers>
 <layer number="1" name="Top" color="4" fill="1" visible="no" active="no"/>
@@
 </segment>
 <segment>
-<pinref part="U1" gate="G$1" pin="PA15"/>
-<wire x1="149.86" y1="198.12" x2="147.32" y2="198.12" width="0.1524" layer="91"/>
-<label x="147.32" y="198.12" size="1.27" layer="95" rot="R180" xref="yes"/>
-</segment>
-<segment>
 <pinref part="8X8_WS2812_BOARD1" gate="G$1" pin="DIN"/>
 <pinref part="8X8_WS2812_BOARD" gate="G$1" pin="DOUT"/>
@@
 <wire x1="96.52" y1="76.2" x2="104.14" y2="76.2" width="0.1524" layer="91"/>
 </segment>
+<segment>
+<pinref part="U1" gate="G$2" pin="PB15"/>
+<wire x1="220.98" y1="165.1" x2="218.44" y2="165.1" width="0.1524" layer="91"/>
+<label x="218.44" y="165.1" size="1.27" layer="95" rot="R180" xref="yes"/>
+</segment>
 </net>
